File: LTC2874_Breakout.kicad_pcb (KiCad board)
At the start: 2 copper layers, 114.3 x 134.6 mm, 86 parts, among them J1 Conn_01x02_Male, J10 Conn_01x03_Male, J11 Conn_01x02_Male, J12 Conn_01x02_Male, J2 Conn_01x04_Male, J3 Conn_01x03_Male, J4 Conn_01x03_Male, J5 Conn_01x03_Male, J6 Conn_01x03_Male, J7 Conn_01x03_Male, J8 Conn_01x03_Male, J9 Conn_01x03_Male, Q1 FQT7N10LTF, Q2 FQT7N10LTF, Q3 FQT7N10LTF, Q4 FQT7N10LTF, U1 LTC2874

Commit message: fix: ライブラリの参照がおかしくなっていた問題を修正 e commit message for your changes. Lines starting
Parts:
- Q1, Q2, Q3, Q4: footprint Package_TO_SOT_SMD:SOT-223-3_TabPin2_empty -> Local:SOT-223-3_TabPin2_empty
- R2, R3, R4, R5: footprint Resistor_SMD:R_0603_1608Metric_Pad0.98x0.95mm_HandSolder -> Resistor_SMD:R_0805_2012Metric_Pad1.20x1.40mm_HandSolder
- U1: footprint Package_SO:TSSOP-38_4.4x9.7mm_P0.5mm_withPad -> Local:TSSOP-38_4.4x9.7mm_P0.5mm_with_Hole
Routing:
- net Net-(D1-Pad2): track 85.2 -> 58.6 mm
- net Net-(D11-Pad1): track 103.7 -> 79.6 mm
- net Net-(D4-Pad1): track 114.8 -> 106.0 mm
- net GND: track 96.4 -> 98.6 mm
Other:
- net class Default removed
- board text added: "2021.7.4 Rev. 0.2"
- board text removed: "2021.6.23 Rev. 0.1"
